Commit message: Patch for go2_nav: back-mounted 3D lidar, RGBD camera, safe roll/pitch handling
- go2_description/package.xml: remove dead gazebo_plugins (Classic Gazebo)
  dependency, unused and unavailable on Jazzy, was blocking rosdep.
- go2_description/xacro/robot.xacro: reposition lidar joint front->back
  mounted, resize its collision cylinder to Livox Mid-360 proportions.
- go2_description/xacro/gazebo.xacro: camera -> rgbd_camera (848x480, 87 HFOV,
  15Hz, 0.2-25m depth clip); lidar upgraded from single-ring 2D scan to a
  real 3D scan (900x40 samples, -7..+52 deg, 0.1-25m); topic renamed
  scan->lidar since gz-sim's raw multi-ring array is no longer a valid 2D
  LaserScan once there's more than one elevation ring.
- quadropted_controller/.../RobotController.py: zero angular.x/angular.y
  (roll/pitch) before they reach the gait controller -- they were never
  meant to be user-commandable and caused continuous non-recovering foot
  drift when held nonzero. linear.z repurposed as a real stance-height
  adjust (was completely dead downstream otherwise).
- go1_description/, docker/: marked COLCON_IGNORE (go1 depends on Classic
  Gazebo packages Jazzy dropped, and isn't used in this project).

Based on go2_ros2_sim_py by abutalipovvv
(https://github.com/abutalipovvv/go2_ros2_sim_py), commit 92d6bc9.

File: go2_description/xacro/gazebo.xacro (robot description, xacro)
@@ -102,8 +102,13 @@
             </sensor>
         </gazebo>
+        <!-- Back-mounted 3D lidar, Livox Mid-360-style FOV (360 x 59 deg, -7..+52 deg
+             elevation). gz-sim's gpu_lidar auto-publishes a flat multi-ring range array
+             on <topic> (not useful once vertical samples > 1) AND a full point cloud on
+             <topic>/points, which is what we actually consume. A separate 2D /scan for
+             SLAM is produced downstream by pointcloud_to_laserscan, not by this sensor
+             directly, hence "lidar" rather than "scan" as the topic base. -->
         <gazebo reference="laser_frame">
-            <!--<material>Gazebo/Black</material>-->
-            <sensor name="laser" type="gpu_lidar">
-                <pose> 0 0 0 0 0 0 </pose>
+            <sensor name="lidar" type="gpu_lidar">
+                <pose>0 0 0 0 0 0</pose>
                 <visualize>false</visualize>
                 <update_rate>10</update_rate>
@@ -111,38 +116,57 @@
                     <scan>
                         <horizontal>
-                            <samples>360</samples>
-                            <min_angle>-3.14</min_angle>
-                            <max_angle>3.14</max_angle>
+                            <samples>900</samples>
+                            <min_angle>-3.14159</min_angle>
+                            <max_angle>3.14159</max_angle>
                         </horizontal>
+                        <vertical>
+                            <samples>40</samples>
+                            <min_angle>-0.12217</min_angle>  <!-- -7 deg -->
+                            <max_angle>0.90757</max_angle>   <!-- +52 deg -->
+                        </vertical>
                     </scan>
                     <range>
-                        <min>0.05</min>
-                        <max>12</max>
+                        <min>0.10</min>
+                        <max>40.0</max>
                     </range>
                 </lidar>
-                <topic>/${robot_name}/scan</topic>
+                <topic>/${robot_name}/lidar</topic>
                 <gz_frame_id>laser_frame</gz_frame_id>
             </sensor>
         </gazebo>
+        <!-- Head-mounted RealSense D435-style RGBD camera, forward-facing (+X).
+             gz-sim's rgbd_camera appends /image, /depth_image, /points, /camera_info
+             to <topic>. -->
         <gazebo reference="camera_face">
-            <!-- <material>Gazebo/Black</material> -->
-            <sensor name="camera" type="camera">
-                <pose> 0 0 0 0 0 0 </pose>
+            <sensor name="camera" type="rgbd_camera">
+                <pose>0 0 0 0 0 0</pose>
                 <visualize>true</visualize>
-                <update_rate>10</update_rate>
+                <update_rate>15</update_rate>
                 <camera>
-                    <camera_info_topic>/${robot_name}/color/camera_info</camera_info_topic>
-                    <horizontal_fov>1.089</horizontal_fov>
+                    <horizontal_fov>1.518</horizontal_fov>  <!-- 87 deg, D435 colour HFOV -->
                     <image>
                         <format>R8G8B8</format>
-                        <width>640</width>
+                        <width>848</width>
                         <height>480</height>
                     </image>
                     <clip>
-                        <near>0.05</near>
-                        <far>8.0</far>
+                        <near>0.10</near>
+                        <far>25.0</far>
                     </clip>
+                    <depth_camera>
+                        <!-- Was 10.0: the office is ~20x20m, so open-room sightlines
+                             routinely exceeded this, returning +Inf for those pixels.
+                             RViz's Image display auto-normalizes min/max over the whole
+                             frame; +Inf in that computation poisons the normalization
+                             constant for every pixel, not just the far ones, which is
+                             why depth rendered fine in small rooms but went blank in
+                             large ones. 25.0 covers the full room diagonal. -->
+                        <clip>
+                            <near>0.20</near>
+                            <far>25.0</far>
+                        </clip>
+                    </depth_camera>
                 </camera>
-                <topic>/${robot_name}/color/image_raw</topic>
+                <topic>/${robot_name}/camera</topic>
                 <gz_frame_id>camera_face</gz_frame_id>
             </sensor>

File: go2_description/xacro/robot.xacro (robot description, xacro)
@@ -57,12 +57,14 @@
         </inertial>
     </link>
+    <!-- Moved to the rear, roof-mounted: was 0.22 0 0.095 (front, near the camera).
+         Requested layout is camera on the head facing forward, lidar on the back. -->
     <joint name='laser_scan' type='fixed'>
-        <parent link="base_link"/>,
+        <parent link="base_link"/>
         <child link="laser_frame"/>
-        <origin xyz="0.22 0.0 0.095" rpy="0 0 0" />
+        <origin xyz="-0.26 0.0 0.14" rpy="0 0 0" />
     </joint>
     <link name="laser_frame">
         <inertial>
-            <mass value="0.001"/>
+            <mass value="0.15"/>
             <origin rpy="0 0 0" xyz="0 0 0"/>
             <inertia ixx="0.0001" ixy="0" ixz="0" iyy="0.0001" iyz="0" izz="0.0001"/>
@@ -71,5 +73,5 @@
             <origin rpy="0 0 0" xyz="0 0 0"/>
             <geometry>
-                <cylinder length="0.01" radius="0.018" />
+                <cylinder length="0.06" radius="0.033" />
             </geometry>
             <!-- <material name="red"/> -->
@@ -78,5 +80,5 @@
             <origin rpy="0 0 0" xyz="0 0 0"/>
             <geometry>
-                <cylinder length="0.01" radius="0.018" />
+                <cylinder length="0.06" radius="0.033" />
             </geometry>
         </collision>
